File: SBK_PFET1/KiCad/SBK_PFET1.kicad_pcb (KiCad board)
At the start: 2 copper layers, 10.7 x 9.9 mm, 4 parts, among them J1 1 x 3 pin header, Q1 AO3401A

Commit message: PFET1 updates
Other:
- board size 10.7 x 9.9 mm -> 10.7 x 10 mm
- board text added: "SBK_PFET1 R1.0"
- board text removed: "SBK_PFET1 v1.0"
