File: SBK_NFET1/KiCad/SBK_NFET1.kicad_pcb (KiCad board)
At the start: 2 copper layers, 10.7 x 9.9 mm, 4 parts, among them J1 1 x 3 pin header, Q1 AO3400A

Commit message: NFET1 updates
Other:
- board size 10.7 x 9.9 mm -> 10.7 x 10 mm
- board text added: "SBK_NFET1 R1.0"
- board text removed: "SBK_NFET1 v1.0"
